File: nRF52832_Base/nRF52832_Base/NRF52832_Base_Reference.sch (KiCad schematic (older format))
At the start: 1 part

Commit message: Added NRF52832 symbol to library and schematic
Parts:
- removed U?: nRF52832-QFxx, Package_DFN_QFN:QFN-48-1EP_6x6mm_P0.4mm_EP4.66x4.66mm, symbol MCU_Nordic:nRF52832-QFxx
- added U?: nRF52832, symbol Project_Libary:nRF52832
Changed lines of the file:
@@
 EESchema Schematic File Version 4
+LIBS:nRF52832_Base-cache
 EELAYER 26 0
 EELAYER END
@@
 $EndDescr
 $Comp
-L MCU_Nordic:nRF52832-QFxx U?
-U 1 1 5B677240
-P 5200 3650
-F 0 "U?" H 5200 1864 50  0000 C CNN
-F 1 "nRF52832-QFxx" H 5200 1773 50  0000 C CNN
-F 2 "Package_DFN_QFN:QFN-48-1EP_6x6mm_P0.4mm_EP4.66x4.66mm" H 5200 1550 50  0001 C CNN
-F 3 "http://infocenter.nordicsemi.com/pdf/nRF52832_PS_v1.4.pdf" H 4700 3850 50  0001 C CNN
-	1    5200 3650
+L Project_Libary:nRF52832 U?
+U 1 1 5B67E14F
+P 5500 4950
+F 0 "U?" H 5750 5800 50  0000 L CNN
+F 1 "nRF52832" H 5600 5650 50  0000 L CNN
+F 2 "" H 5500 4950 50  0001 C CNN
+F 3 "" H 5500 4950 50  0001 C CNN
+	1    5500 4950
 	1    0    0    -1
 $EndComp
