File: Motor_4_Channel_V2/Motor_4_Channel_V2.kicad_pcb (KiCad board)
At the start: 2 copper layers, 100 x 100 mm, 90 parts, among them J1 Conn_01x02_Male, J10 Conn_01x02_Male, J11 Conn_01x10_Male, J2 Conn_01x02_Male, J3 Conn_01x02_Male, J4 Conn_01x02_Male, J5 Conn_01x02_Male, J6 Conn_01x02_Male, J7 Conn_01x02_Male, J8 Conn_01x10_Male, J9 Conn_01x02_Male, K1 G8N-1L-DC12, K2 G8N-1L-DC12, K3 G8N-1L-DC12, K4 G8N-1L-DC12, P1 Pad, P10 Pad, P11 Pad, P12 Pad, P2 Pad, P3 Pad, P4 Pad, P5 Pad, P6 Pad, P7 Pad, P8 Pad, P9 Pad, Q1 Q_NMOS_GDS, Q2 Q_NMOS_GDS, Q3 Q_NMOS_GDS, Q4 Q_NMOS_GDS, Q5 Q_NMOS_GDS, Q6 Q_NMOS_GDS, Q7 Q_NMOS_GDS, Q8 Q_NMOS_GDS, SW1 SW_SPST, U1 SN74LVC1G139DCUR, U10 NC7WZ14P6XCT-ND, U11 MSP430G2553_LP, U12 G8NW-2H-DC12, U13 G8NW-2H-DC12, U14 G8NW-2H-DC12, U15 G8NW-2H-DC12, U2 SN74LVC1G139DCUR, U3 UA78M05IDCY, U4 UA78M33QDCYRG4Q1, U5 NC7WZ14P6XCT-ND, U6 NC7WZ14P6XCT-ND, U7 SN74LVC1G139DCUR, U8 SN74LVC1G139DCUR, U9 NC7WZ14P6XCT-ND

Commit message: Switched THT 2-pin male headers for buttons and led with SMT headers. Rearranged SMT components,
Parts:
- D11, D2, D5, D8, Q1, Q2, Q3, Q4, Q5, Q6, Q7, Q8, R13, R14, R15, R16, R17, R18, R19, R20, U1, U10, U2, U5, U6, U7, U8, U9: moved to F.Cu
- J1, J10, J2, J3, J4, J5, J6, J7, J9: footprint Connector_PinHeader_2.54mm:PinHeader_1x02_P2.54mm_Vertical -> Connector_PinHeader_2.54mm:PinHeader_1x02_P2.54mm_Vertical_SMD_Pin1Left
- moved J5 19.4 mm to (137.4, 106.2)
- moved J6 19.2 mm to (182.4, 106.6)
- moved J4 19.1 mm to (160.0, 106.3)
- moved J3 18.8 mm to (114.0, 106.2)
- moved R2 15.8 mm to (95.2, 105.9), turned to 270 degrees
- moved J9 14.7 mm to (170.3, 106.2)
- moved J7 14.5 mm to (147.4, 106.2)
- moved R9 14.5 mm to (173.2, 110.4)
- moved J2 14.4 mm to (124.3, 106.2)
- moved R3 13.9 mm to (127.0, 110.2)
- moved R5 13.9 mm to (150.0, 110.2)
- moved J1 13.5 mm to (99.8, 106.2)
- moved R1 12.7 mm to (102.6, 110.1)
- moved R6 12.1 mm to (144.5, 102.0), turned to 180 degrees
- moved R4 12.1 mm to (121.3, 102.1), turned to 180 degrees
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Connections:
- J11 pad 1: OUT_2 -> DIR_2
- J11 pad 2: DIR_2 -> OUT_2
- J11 pad 4: OUT_3 -> DIR_3
- J11 pad 5: DIR_3 -> OUT_3
- J11 pad 7: OUT_4 -> DIR_4
- J11 pad 8: DIR_4 -> OUT_4
- J8 pad 1: OUT_1 -> DIR_1
- J8 pad 2: DIR_1 -> OUT_1
- U11 pad 10: OUT_2 -> DIR_2
- U11 pad 11: OUT_1 -> DIR_1
- U11 pad 12: DIR_1 -> OUT_1
- U11 pad 3: DIR_4 -> OUT_4
- U11 pad 4: OUT_4 -> DIR_4
- U11 pad 6: DIR_3 -> OUT_3
- U11 pad 7: OUT_3 -> DIR_3
- U11 pad 9: DIR_2 -> OUT_2
Routing:
- net 5V_REF: track 163.8 -> 212.5 mm, vias 5 -> 16
- net BTN_2: track 56.4 -> 26.8 mm, vias 1 -> 0
- net GND: track 72.4 -> 48.1 mm, vias 115 -> 99
- net BTN_1: track 79.0 -> 56.2 mm, vias 2 -> 0
- net OUT_2: track 73.1 -> 50.9 mm, vias 1 -> 0
- net 12V_REF: track 525.9 -> 505.9 mm, vias 8 -> 9
- net BTN_3: track 54.3 -> 34.9 mm, vias 2 -> 1
- net RED_4: track 7.94 -> 25.9 mm
- net DIR_2: track 78.5 -> 60.7 mm, vias 3 -> 2
- net RED_2: track 7.69 -> 25.2 mm
- net RED_3: track 7.89 -> 24.6 mm
- net DIR_1: track 102.2 -> 89.0 mm, vias 5 -> 2
- net RED_1: track 7.89 -> 20.9 mm
- net OUT_3: track 44.2 -> 32.7 mm
- net SW4_CTL: track 12.6 -> 21.9 mm
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- added copper zone on B.Cu, net V+

Commit message: Misc. changes to Motor PCB.
Parts:
- added C10: 0.1uF, Capacitor_SMD:C_0603_1608Metric_Pad1.05x0.95mm_HandSolder, F.Cu at (200.4, 122.9)
- added C8: 0.1uF, Capacitor_SMD:C_0603_1608Metric_Pad1.05x0.95mm_HandSolder, F.Cu at (197.0, 122.9)
- added C9: 0.1uF, Capacitor_SMD:C_0603_1608Metric_Pad1.05x0.95mm_HandSolder, F.Cu at (197.0, 124.4)
- R2, R4, R6: value R -> 47k
Connections:
- J1 pad 2: RED_1 -> Net-(J1-Pad2)
- J2 pad 2: RED_2 -> Net-(J2-Pad2)
- J3 pad 1: GND -> BTN_1
- J3 pad 2: BTN_1 -> GND
- J4 pad 1: GND -> BTN_3
- J4 pad 2: BTN_3 -> GND
- J5 pad 1: GND -> BTN_2
- J5 pad 2: BTN_2 -> GND
- J6 pad 1: GND -> BTN_4
- J6 pad 2: BTN_4 -> GND
- J7 pad 2: RED_3 -> Net-(J7-Pad2)
- J9 pad 2: RED_4 -> Net-(J9-Pad2)
- K1 pad 2: 12V_REF -> SW1_CTL
- K1 pad 5: SW1_CTL -> 12V_REF
- K2 pad 2: 12V_REF -> SW2_CTL
- K2 pad 5: SW2_CTL -> 12V_REF
- K3 pad 2: 12V_REF -> SW3_CTL
- K3 pad 5: SW3_CTL -> 12V_REF
- K4 pad 2: 12V_REF -> SW4_CTL
- K4 pad 5: SW4_CTL -> 12V_REF
- P10 pad 1: /Sheet5C130375/OUT_3- -> /Sheet5C130375/OUT_3+
- P11 pad 1: /Sheet5C130375/OUT_4+ -> /Sheet5C130375/OUT_4-
- P12 pad 1: /Sheet5C130375/OUT_4- -> /Sheet5C130375/OUT_4+
- P5 pad 1: /Sheet5C130375/OUT_1+ -> /Sheet5C130375/OUT_1-
- P6 pad 1: /Sheet5C130375/OUT_1- -> /Sheet5C130375/OUT_1+
- P7 pad 1: /Sheet5C130375/OUT_2+ -> /Sheet5C130375/OUT_2-
- P8 pad 1: /Sheet5C130375/OUT_2- -> /Sheet5C130375/OUT_2+
- P9 pad 1: /Sheet5C130375/OUT_3+ -> /Sheet5C130375/OUT_3-
- R1 pad 1: RED_1 -> Net-(J1-Pad2)
- R1 pad 2: GND -> RED_1
- R12 pad 1: BTN_3 -> 3V3_REF
- R12 pad 2: 3V3_REF -> BTN_3
- R2 pad 1: GREEN_1 -> 3V3_REF
- R2 pad 2: GND -> BTN_1
- R3 pad 1: RED_2 -> Net-(J2-Pad2)
- R3 pad 2: GND -> RED_2
- R4 pad 1: GREEN_2 -> 3V3_REF
- R4 pad 2: GND -> BTN_2
- R5 pad 1: RED_3 -> Net-(J7-Pad2)
- R5 pad 2: GND -> RED_3
- R6 pad 1: GREEN_3 -> 3V3_REF
- R6 pad 2: GND -> BTN_4
- R9 pad 1: RED_4 -> Net-(J9-Pad2)
- R9 pad 2: GND -> RED_4
- U12 pad 1: /Sheet5C130375/OUT_1- -> /Sheet5C130375/OUT_1+
- U12 pad 6: /Sheet5C130375/OUT_1+ -> /Sheet5C130375/OUT_1-
- U13 pad 1: /Sheet5C130375/OUT_2- -> /Sheet5C130375/OUT_2+
- U13 pad 6: /Sheet5C130375/OUT_2+ -> /Sheet5C130375/OUT_2-
- U14 pad 1: /Sheet5C130375/OUT_3- -> /Sheet5C130375/OUT_3+
- U14 pad 6: /Sheet5C130375/OUT_3+ -> /Sheet5C130375/OUT_3-
- U15 pad 1: /Sheet5C130375/OUT_4- -> /Sheet5C130375/OUT_4+
- U15 pad 6: /Sheet5C130375/OUT_4+ -> /Sheet5C130375/OUT_4-
Routing:
- net Net-(K3-Pad3): track 22.6 -> 0.00 mm
- net Net-(K4-Pad3): track 22.5 -> 0.03 mm
- net Net-(K1-Pad3): track 21.2 -> 24.5 mm
- net GND: track 48.1 -> 45.3 mm, vias 99 -> 96
- net RED_1: track 20.9 -> 22.3 mm, vias 0 -> 1
- net BTN_1: track 56.2 -> 57.6 mm, vias 0 -> 1
- net Net-(K2-Pad4): track 0.00 -> 1.11 mm
- net /Sheet5C130375/OUT_4-: track 10.4 -> 9.53 mm
- net /Sheet5C130375/OUT_4+: track 9.53 -> 10.4 mm
