File: Buck_Converter_V1/Buck_Converter_V1.sch (KiCad schematic (older format))
At the start: 17 parts

Commit message: Finished schematic. Changed compensation to Type 3. Added fuse to input. Finished adding values and footprints for all components.
Parts:
- removed R?: R, symbol Device:R
- removed R?: 25k, symbol Device:R
- added C8: 4.7nF, Capacitor_SMD:C_0603_1608Metric_Pad1.05x0.95mm_HandSolder, symbol Device:C
- added F1: Fuse, Fuse:Fuse_0603_1608Metric_Pad1.05x0.95mm_HandSolder, symbol Device:Fuse
- added J1, J2, J3, J4: Conn_01x01_Male, Connector_PinHeader_2.54mm:PinHeader_1x01_P2.54mm_Vertical, symbol Connector:Conn_01x01_Male
- added R5: 383, Resistor_SMD:R_0603_1608Metric_Pad1.05x0.95mm_HandSolder, symbol Device:R
- added RV1: 25k, Potentiometer_THT:Potentiometer_Bourns_3296W_Vertical, symbol Device:R_POT_TRIM
- added RV2: 4125, Potentiometer_THT:Potentiometer_Bourns_3296W_Vertical, symbol Device:R_POT_TRIM
- C1, C3, C4: renamed from C?; footprint (none) -> Capacitor_SMD:C_0603_1608Metric_Pad1.05x0.95mm_HandSolder
- C2: renamed from C?; value 100uF -> 180uF; footprint (none) -> Custom_Footprints:C_AlPo_Radial_SMT_8.3mmx8.3mm
- C5: renamed from C?; value C -> 6.8nF; footprint (none) -> Capacitor_SMD:C_0603_1608Metric_Pad1.05x0.95mm_HandSolder
- C6: renamed from C?; value C -> 180uF; footprint (none) -> Custom_Footprints:C_AlPo_Radial_SMT_8.3mmx8.3mm
- C7: renamed from C?; value C -> 68pF; footprint (none) -> Capacitor_SMD:C_0603_1608Metric_Pad1.05x0.95mm_HandSolder
- D1: renamed from D?; value D_Schottky -> NRVTSA4100ET3G; footprint (none) -> Diode_SMD:D_SMA_Handsoldering
- L1: renamed from L?; value L -> 33uH; footprint (none) -> Inductor_SMD:L_12x12mm_H8mm
- Q1: renamed from Q?; value Q_PMOS_GSD -> SI2319CDS-T1-GE3; footprint (none) -> Package_TO_SOT_SMD:SOT-23
- R1, R2: renamed from R?; footprint (none) -> Resistor_SMD:R_0603_1608Metric_Pad1.05x0.95mm_HandSolder
- R3: renamed from R?; value R -> 14.9k; footprint (none) -> Resistor_SMD:R_0603_1608Metric_Pad1.05x0.95mm_HandSolder
- R4: renamed from R?; value R -> 16.5k; footprint (none) -> Resistor_SMD:R_0603_1608Metric_Pad1.05x0.95mm_HandSolder
- U1: renamed from U?; footprint (none) -> Package_SO:SOIC-8_3.9x4.9mm_P1.27mm
Connections:
- net GND: now also J2.1 (Pin_1), J4.1 (Pin_1), RV1.1, RV2.2
- net Vin: now also F1.1
- net Vout: now also C8.1, J3.1 (Pin_1)
- net at C7.1, R3.1, R4.2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: now also R5.2, RV2.3
- net at U1.7 (RT): now also RV1.2
- new net: C8.2, R5.1
- new net: F1.2, J1.1 (Pin_1)
- no-connect marks 0 -> 2
Other:
- note added: "Power input and output. Extra pads will be added in the PCB layout to solder wires instead"
- moved on the sheet: R4
