File: Buck_Converter_V1/Buck_Converter_V1.sch (KiCad schematic (older format))
At the start: 24 parts, among them J1 Conn_01x01_Male, J2 Conn_01x01_Male, J3 Conn_01x01_Male, J4 Conn_01x01_Male, Q1 SI2319CDS-T1-GE3, U1 TL5001CDR

Commit message: Changed footprint for PMOS switch. Generated gerber files.
Parts:
- Q1: footprint Package_TO_SOT_SMD:SOT-23 -> Package_TO_SOT_SMD:SOT-23_Handsoldering
Changed lines of the file:
@@
 F 0 "Q1" V 2125 1725 50  0000 C CNN
 F 1 "SI2319CDS-T1-GE3" V 2216 1725 50  0001 C CNN
-F 2 "Package_TO_SOT_SMD:SOT-23" H 2075 1825 50  0001 C CNN
+F 2 "Package_TO_SOT_SMD:SOT-23_Handsoldering" H 2075 1825 50  0001 C CNN
 F 3 "~" H 1875 1725 50  0001 C CNN
 	1    1875 1725

Commit message: Updating branch
Parts:
- U1: symbol Project_Libary:TL5001CDR -> Buck_Converter_V1-rescue:TL5001CDR-Project_Libary
Changed lines of the file:
@@
 P_DRIVE
 $Comp
-L Project_Libary:TL5001CDR U1
+L Buck_Converter_V1-rescue:TL5001CDR-Project_Libary U1
 U 1 1 5C189351
 P 1950 3700
