File: Outlet_Relay_V1/Outlet_Relay_V1.sch (KiCad schematic (older format))
At the start: 7 parts

Commit message: Set footprints for flyback diode and mosfet
Parts:
- D?: footprint (none) -> Diode_SMD:D_SOD-123F
- Q?: value Q_NMOS_GDS -> Q_NMOS_GSD; footprint (none) -> Package_TO_SOT_SMD:SOT-23_Handsoldering
Changed lines of the file:
@@
 P 4975 3800
 F 0 "Q?" H 5180 3846 50  0000 L CNN
-F 1 "Q_NMOS_GDS" H 5180 3755 50  0000 L CNN
-F 2 "" H 5175 3900 50  0001 C CNN
+F 1 "Q_NMOS_GSD" H 5180 3755 50  0000 L CNN
+F 2 "Package_TO_SOT_SMD:SOT-23_Handsoldering" H 5175 3900 50  0001 C CNN
 F 3 "~" H 4975 3800 50  0001 C CNN
 	1    4975 3800
@@
 F 0 "D?" V 5029 3204 50  0000 L CNN
 F 1 "D" V 5120 3204 50  0000 L CNN
-F 2 "" H 5075 3125 50  0001 C CNN
+F 2 "Diode_SMD:D_SOD-123F" H 5075 3125 50  0001 C CNN
 F 3 "~" H 5075 3125 50  0001 C CNN
 	1    5075 3125
