File: NRF52832_Reference/NRF52832_Reference.sch (KiCad schematic (older format))
At the start: 53 parts, among them J1 Conn_01x10_Male, J10 Conn_01x10_Male, J11 Conn_01x04_Male, J12 SWD_Header, J13 Conn_01x02_Male, J14 Conn_01x02_Male, J15 Conn_01x02_Male, J2 Conn_01x10_Male, J3 Conn_01x02_Male, J4 Conn_01x02_Male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

Commit message: Updated component placement for PCB layout
Parts:
- removed J13, J14, J15, J8, J9: Conn_01x02_Male, Connector_PinHeader_2.54mm:PinHeader_1x02_P2.54mm_Vertical, symbol Connector:Conn_01x02_Male
- R3, R4: value 10k -> 4.7k
Connections:
- net P0.11_SDA: now also R3.2, U2.5 (SDA), U4.3 (SDA), U5.1 (SDA)
- net P0.12_SCL: now also R4.2, U2.6 (SCL), U4.4 (SCL), U5.2 (SCL)
- net P0.22: now also R11.1
- net P0.23: now also R8.1
Changed lines of the file:
@@
 P 5275 7000
 F 0 "R3" H 5345 7046 50  0000 L CNN
-F 1 "10k" H 5345 6955 50  0000 L CNN
+F 1 "4.7k" H 5345 6955 50  0000 L CNN
 F 2 "Resistor_SMD:R_0603_1608Metric_Pad1.05x0.95mm_HandSolder" V 5205 7000 50  0001 C CNN
 F 3 "~" H 5275 7000 50  0001 C CNN
@@
 P 5575 7000
 F 0 "R4" H 5645 7046 50  0000 L CNN
-F 1 "10k" H 5645 6955 50  0000 L CNN
+F 1 "4.7k" H 5645 6955 50  0000 L CNN
 F 2 "Resistor_SMD:R_0603_1608Metric_Pad1.05x0.95mm_HandSolder" V 5505 7000 50  0001 C CNN
 F 3 "~" H 5575 7000 50  0001 C CNN
@@
 	1    0    0    -1
 $EndComp
-$Comp
-L Connector:Conn_01x02_Male J8
-U 1 1 5C0A43EB
-P 5950 7050
-F 0 "J8" V 6056 7091 50  0000 L CNN
-F 1 "Conn_01x02_Male" V 6101 7090 50  0001 L CNN
-F 2 "Connector_PinHeader_2.54mm:PinHeader_1x02_P2.54mm_Vertical" H 5950 7050 50  0001 C CNN
-F 3 "~" H 5950 7050 50  0001 C CNN
-	1    5950 7050
-	0    1    1    0
-$EndComp
-$Comp
-L Connector:Conn_01x02_Male J9
-U 1 1 5C0A458E
-P 5950 7700
-F 0 "J9" V 6025 7525 50  0000 R CNN
-F 1 "Conn_01x02_Male" V 6012 7513 50  0001 R CNN
-F 2 "Connector_PinHeader_2.54mm:PinHeader_1x02_P2.54mm_Vertical" H 5950 7700 50  0001 C CNN
-F 3 "~" H 5950 7700 50  0001 C CNN
-	1    5950 7700
-	0    1    -1   0
-$EndComp
-Wire Wire Line
-	6075 7300 5950 7300
-Wire Wire Line
-	5950 7300 5950 7250
-Wire Wire Line
-	6075 7425 5950 7425
-Wire Wire Line
-	5950 7425 5950 7500
 Wire Wire Line
 	3775 6600 3925 6600
@@
 Connection ~ 5275 5850
 Wire Wire Line
-	5850 7250 5850 7300
-Wire Wire Line
-	5850 7300 5575 7300
-Wire Wire Line
 	4475 7300 4475 6850
 Wire Wire Line
@@
 	1725 7300 1725 6850
 Connection ~ 3050 7300
-Wire Wire Line
-	5850 7500 5850 7425
-Wire Wire Line
-	5850 7425 5275 7425
 Wire Wire Line
 	4375 7425 4375 6850
@@
 	0    -1   -1   0
 $EndComp
-$Comp
-L Connector:Conn_01x02_Male J13
-U 1 1 5C284A46
-P 9100 1525
-F 0 "J13" H 9072 1451 50  0000 R CNN
-F 1 "Conn_01x02_Male" H 9206 1612 50  0001 C CNN
-F 2 "Connector_PinHeader_2.54mm:PinHeader_1x02_P2.54mm_Vertical" H 9100 1525 50  0001 C CNN
-F 3 "~" H 9100 1525 50  0001 C CNN
-	1    9100 1525
-	-1   0    0    1
-$EndComp
-$Comp
-L Connector:Conn_01x02_Male J14
-U 1 1 5C284AEA
-P 9800 1525
-F 0 "J14" H 9772 1451 50  0000 R CNN
-F 1 "Conn_01x02_Male" H 9906 1612 50  0001 C CNN
-F 2 "Connector_PinHeader_2.54mm:PinHeader_1x02_P2.54mm_Vertical" H 9800 1525 50  0001 C CNN
-F 3 "~" H 9800 1525 50  0001 C CNN
-	1    9800 1525
-	-1   0    0    1
-$EndComp
 Text GLabel 7850 675  0    50   Input ~ 0
 3V3_Ref
@@
 	10050 1275 8425 1275
 Connection ~ 8425 1275
-Wire Wire Line
-	8900 1425 8900 1175
 Connection ~ 8900 1175
 Wire Wire Line
 	8900 1175 7750 1175
-Wire Wire Line
-	9600 1425 9600 1075
 Connection ~ 9600 1075
 Wire Wire Line
@@
 Text Notes 3900 650  0    50   ~ 0
 GPIO and Button/LEDs
-$Comp
-L Connector:Conn_01x02_Male J15
-U 1 1 5C377AB0
-P 10925 3775
-F 0 "J15" H 10897 3701 50  0000 R CNN
-F 1 "Conn_01x02_Male" H 10898 3746 50  0001 R CNN
-F 2 "Connector_PinHeader_2.54mm:PinHeader_1x02_P2.54mm_Vertical" H 10925 3775 50  0001 C CNN
-F 3 "~" H 10925 3775 50  0001 C CNN
-	1    10925 3775
-	-1   0    0    1
-$EndComp
-Wire Wire Line
-	10725 3675 10075 3675
-Wire Wire Line
-	10075 3675 10075 3600
-Wire Wire Line
-	10725 3775 10200 3775
-Wire Wire Line
-	10200 3775 10200 3500
-Text Label 10300 3675 0    50   ~ 0
+Text Label 9700 3600 0    50   ~ 0
 SWDCLK
-Text Label 10300 3775 0    50   ~ 0
+Text Label 9800 3500 0    50   ~ 0
 SWDIO
 Connection ~ 4000 3075
@@
 P 4775 1450
 F 0 "J2" H 4881 2028 50  0000 C CNN
-F 1 "Conn_01x10_Male" H 4881 1937 50  0000 C CNN
+F 1 "Conn_01x10_Male" H 4881 1937 50  0001 C CNN
 F 2 "Connector_PinHeader_2.54mm:PinHeader_1x10_P2.54mm_Vertical" H 4775 1450 50  0001 C CNN
 F 3 "~" H 4775 1450 50  0001 C CNN
@@
 U 1 1 5C1BC35E
 P 10075 4025
-F 0 "R14" H 9900 4075 50  0000 L CNN
+F 0 "R14" H 9875 4075 50  0000 L CNN
 F 1 "22" H 9925 3975 50  0000 L CNN
 F 2 "Resistor_SMD:R_0603_1608Metric_Pad1.05x0.95mm_HandSolder" V 10005 4025 50  0001 C CNN
@@
 	10200 4175 10200 5100
 Wire Wire Line
-	10075 3875 10075 3675
-Connection ~ 10075 3675
-Wire Wire Line
-	10200 3875 10200 3775
-Connection ~ 10200 3775
+	10075 3600 10075 3875
+Wire Wire Line
+	10200 3500 10200 3875
+Wire Wire Line
+	5575 7300 6075 7300
+Wire Wire Line
+	5275 7425 6075 7425
+Wire Wire Line
+	8900 1175 8900 1525
+Wire Wire Line
+	9600 1075 9600 1525
 $EndSCHEMATC

Commit message: Finished component placement on PCB layout. Ready for routing.
Connections:
- net SWDCLK: no longer names the net of J12.4 (Pin_4), R14.1
- net SWDIO: no longer names the net of J12.2 (Pin_2), R15.1, R9.2
Changed lines of the file:
@@
 Text Notes 3900 650  0    50   ~ 0
 GPIO and Button/LEDs
-Text Label 9700 3600 0    50   ~ 0
-SWDCLK
-Text Label 9800 3500 0    50   ~ 0
-SWDIO
 Connection ~ 4000 3075
 Connection ~ 4000 3750

Commit message: Finished routing of components. Silkscreen labels still not finished.
Connections:
- net 3V3_Ref: now also J1.9 (Pin_9), U1.3; no longer J1.3 (Pin_3), U1.4
- net 3V_Ref: now also U1.6; no longer U1.1
- net 5V_Ref: now also J1.10 (Pin_10); no longer J1.2 (Pin_2)
- net P0.02: now also J2.9 (Pin_9); no longer J2.1 (Pin_1)
- net P0.03: now also J2.8 (Pin_8); no longer J2.2 (Pin_2)
- net P0.04: now also J2.7 (Pin_7), R11.1; no longer J2.3 (Pin_3)
- net P0.05: now also J2.6 (Pin_6), R8.1; no longer J2.4 (Pin_4)
- net P0.07_RES: now also J2.4 (Pin_4); no longer J2.6 (Pin_6)
- net P0.08_A0: now also J2.3 (Pin_3); no longer J2.7 (Pin_7)
- net P0.09_SCL: now also J2.2 (Pin_2); no longer J2.8 (Pin_8)
- net P0.10_SI: now also J2.1 (Pin_1); no longer J2.9 (Pin_9)
- net P0.22: no longer R11.1
- net P0.23: no longer R8.1
- net P0.25: now also J1.2 (Pin_2); no longer J1.4 (Pin_4)
- net P0.26: now also J1.3 (Pin_3); no longer J1.5 (Pin_5)
- net P0.27: now also J1.4 (Pin_4); no longer J1.6 (Pin_6)
- net P0.28: now also J1.5 (Pin_5); no longer J1.7 (Pin_7)
- net P0.29: now also J1.6 (Pin_6); no longer J1.8 (Pin_8)
- net P0.30: now also J1.7 (Pin_7); no longer J1.9 (Pin_9)
- net P0.31: now also J1.8 (Pin_8); no longer J1.10 (Pin_10)
- net Sheet5BF15571/SWDCLK: no longer R13.1
- net at J12.4 (Pin_4), R14.1: now also R13.1
- net at R1.1, R2.1, U3.12 (VDD): now also U1.2; no longer U1.5
- net at U3.18 (A): now also U1.5; no longer U1.2
Other:
- moved on the sheet: D1, D2, R11, R14, R15, R8
Changed lines of the file:
@@
 F 3 "" H 1200 3350 50  0001 C CNN
 	1    1200 3100
-	1    0    0    -1
+	-1   0    0    1
 $EndComp
 NoConn ~ 1300 3275
@@
 Wire Wire Line
 	5650 4225 5275 4225
-Text GLabel 3825 1175 2    50   Input ~ 0
+Text GLabel 3825 1975 2    50   Input ~ 0
 5V_Ref
-Text GLabel 3825 1275 2    50   Input ~ 0
+Text GLabel 3825 1875 2    50   Input ~ 0
 3V3_Ref
+Text GLabel 3825 1175 2    50   BiDi ~ 0
+P0.25
+Text GLabel 3825 1275 2    50   BiDi ~ 0
+P0.26
 Text GLabel 3825 1375 2    50   BiDi ~ 0
-P0.25
+P0.27
 Text GLabel 3825 1475 2    50   BiDi ~ 0
-P0.26
+P0.28
 Text GLabel 3825 1575 2    50   BiDi ~ 0
-P0.27
+P0.29
 Text GLabel 3825 1675 2    50   BiDi ~ 0
-P0.28
+P0.30
 Text GLabel 3825 1775 2    50   BiDi ~ 0
-P0.29
-Text GLabel 3825 1875 2    50   BiDi ~ 0
-P0.30
-Text GLabel 3825 1975 2    50   BiDi ~ 0
 P0.31
 Text Notes 1200 2725 0    50   ~ 0
@@
 Wire Notes Line
 	6950 2575 6950 7775
-Text GLabel 4975 1050 2    50   BiDi ~ 0
+Text GLabel 4975 1850 2    50   BiDi ~ 0
 P0.02
-Text GLabel 4975 1150 2    50   BiDi ~ 0
+Text GLabel 4975 1750 2    50   BiDi ~ 0
 P0.03
-Text GLabel 4975 1250 2    50   BiDi ~ 0
+Text GLabel 4975 1650 2    50   BiDi ~ 0
 P0.04
-Text GLabel 4975 1350 2    50   BiDi ~ 0
+Text GLabel 4975 1550 2    50   BiDi ~ 0
 P0.05
 Text GLabel 4975 1450 2    50   BiDi ~ 0
 P0.06_CS1
-Text GLabel 4975 1550 2    50   BiDi ~ 0
+Text GLabel 4975 1350 2    50   BiDi ~ 0
 P0.07_RES
-Text GLabel 4975 1650 2    50   BiDi ~ 0
+Text GLabel 4975 1250 2    50   BiDi ~ 0
 P0.08_A0
-Text GLabel 4975 1750 2    50   BiDi ~ 0
+Text GLabel 4975 1150 2    50   BiDi ~ 0
 P0.09_SCL
-Text GLabel 4975 1850 2    50   BiDi ~ 0
+Text GLabel 4975 1050 2    50   BiDi ~ 0
 P0.10_SI
-Text GLabel 6250 1050 2    50   BiDi ~ 0
-P0.11_SDA
-Text GLabel 6250 1150 2    50   BiDi ~ 0
-P0.12_SCL
 Text GLabel 6250 1250 2    50   BiDi ~ 0
 P0.13
@@
 L Device:R R8
 U 1 1 5C284626
-P 8900 1675
-F 0 "R8" H 8970 1721 50  0000 L CNN
-F 1 "100" H 8970 1630 50  0000 L CNN
-F 2 "Resistor_SMD:R_0603_1608Metric_Pad1.05x0.95mm_HandSolder" V 8830 1675 50  0001 C CNN
-F 3 "~" H 8900 1675 50  0001 C CNN
-	1    8900 1675
+P 9725 1625
+F 0 "R8" H 9795 1671 50  0000 L CNN
+F 1 "100" H 9795 1580 50  0000 L CNN
+F 2 "Resistor_SMD:R_0603_1608Metric_Pad1.05x0.95mm_HandSolder" V 9655 1625 50  0001 C CNN
+F 3 "~" H 9725 1625 50  0001 C CNN
+	1    9725 1625
 	1    0    0    -1
 $EndComp
@@
 L Device:R R11
 U 1 1 5C2846C2
-P 9600 1675
-F 0 "R11" H 9670 1721 50  0000 L CNN
-F 1 "100" H 9670 1630 50  0000 L CNN
-F 2 "Resistor_SMD:R_0603_1608Metric_Pad1.05x0.95mm_HandSolder" V 9530 1675 50  0001 C CNN
-F 3 "~" H 9600 1675 50  0001 C CNN
-	1    9600 1675
+P 10425 1625
+F 0 "R11" H 10495 1671 50  0000 L CNN
+F 1 "100" H 10495 1580 50  0000 L CNN
+F 2 "Resistor_SMD:R_0603_1608Metric_Pad1.05x0.95mm_HandSolder" V 10355 1625 50  0001 C CNN
+F 3 "~" H 10425 1625 50  0001 C CNN
+	1    10425 1625
 	1    0    0    -1
 $EndComp
@@
 L Device:LED D1
 U 1 1 5C2847C2
-P 8900 1975
-F 0 "D1" V 8938 1858 50  0000 R CNN
-F 1 "LED" V 8847 1858 50  0000 R CNN
-F 2 "LED_SMD:LED_0603_1608Metric_Pad1.05x0.95mm_HandSolder" H 8900 1975 50  0001 C CNN
-F 3 "~" H 8900 1975 50  0001 C CNN
-	1    8900 1975
+P 9725 1925
+F 0 "D1" V 9763 1808 50  0000 R CNN
+F 1 "LED" V 9672 1808 50  0000 R CNN
+F 2 "LED_SMD:LED_0603_1608Metric_Pad1.05x0.95mm_HandSolder" H 9725 1925 50  0001 C CNN
+F 3 "~" H 9725 1925 50  0001 C CNN
+	1    9725 1925
 	0    -1   -1   0
 $EndComp
@@
 L Device:LED D2
 U 1 1 5C28496C
-P 9600 1975
-F 0 "D2" V 9638 1858 50  0000 R CNN
-F 1 "LED" V 9547 1858 50  0000 R CNN
-F 2 "LED_SMD:LED_0603_1608Metric_Pad1.05x0.95mm_HandSolder" H 9600 1975 50  0001 C CNN
-F 3 "~" H 9600 1975 50  0001 C CNN
-	1    9600 1975
+P 10425 1925
+F 0 "D2" V 10463 1808 50  0000 R CNN
+F 1 "LED" V 10372 1808 50  0000 R CNN
+F 2 "LED_SMD:LED_0603_1608Metric_Pad1.05x0.95mm_HandSolder" H 10425 1925 50  0001 C CNN
+F 3 "~" H 10425 1925 50  0001 C CNN
+	1    10425 1925
 	0    -1   -1   0
 $EndComp
 Text GLabel 7850 675  0    50   Input ~ 0
 3V3_Ref
-Text GLabel 10050 1075 2    50   BiDi ~ 0
+Text GLabel 7750 1075 2    50   BiDi ~ 0
 P0.22
-Text GLabel 10050 1175 2    50   BiDi ~ 0
+Text GLabel 7750 1175 2    50   BiDi ~ 0
 P0.23
-Text GLabel 10050 1275 2    50   BiDi ~ 0
+Text GLabel 8775 1275 2    50   BiDi ~ 0
 P0.24
-Wire Wire Line
-	10050 1075 9600 1075
-Wire Wire Line
-	10050 1175 8900 1175
-Wire Wire Line
-	10050 1275 8425 1275
-Connection ~ 8425 1275
-Connection ~ 8900 1175
-Wire Wire Line
-	8900 1175 7750 1175
-Connection ~ 9600 1075
-Wire Wire Line
-	9600 1075 7750 1075
 Wire Wire Line
 	8025 1275 8025 975
@@
 L power:GND #PWR0114
 U 1 1 5C307A96
-P 8900 2200
-F 0 "#PWR0114" H 8900 1950 50  0001 C CNN
-F 1 "GND" H 8905 2027 50  0000 C CNN
-F 2 "" H 8900 2200 50  0001 C CNN
-F 3 "" H 8900 2200 50  0001 C CNN
-	1    8900 2200
+P 9725 2150
+F 0 "#PWR0114" H 9725 1900 50  0001 C CNN
+F 1 "GND" H 9730 1977 50  0000 C CNN
+F 2 "" H 9725 2150 50  0001 C CNN
+F 3 "" H 9725 2150 50  0001 C CNN
+	1    9725 2150
 	1    0    0    -1
 $EndComp
@@
 L power:GND #PWR0115
 U 1 1 5C307B03
-P 9600 2200
-F 0 "#PWR0115" H 9600 1950 50  0001 C CNN
-F 1 "GND" H 9605 2027 50  0000 C CNN
-F 2 "" H 9600 2200 50  0001 C CNN
-F 3 "" H 9600 2200 50  0001 C CNN
-	1    9600 2200
-	1    0    0    -1
-$EndComp
-Wire Wire Line
-	8900 2125 8900 2200
-Wire Wire Line
-	9600 2125 9600 2200
+P 10425 2150
+F 0 "#PWR0115" H 10425 1900 50  0001 C CNN
+F 1 "GND" H 10430 1977 50  0000 C CNN
+F 2 "" H 10425 2150 50  0001 C CNN
+F 3 "" H 10425 2150 50  0001 C CNN
+	1    10425 2150
+	1    0    0    -1
+$EndComp
+Wire Wire Line
+	9725 2075 9725 2150
+Wire Wire Line
+	10425 2075 10425 2150
 Wire Notes Line
 	475  2575 11225 2575
@@
 L Device:R R14
 U 1 1 5C1BC35E
-P 10075 4025
-F 0 "R14" H 9875 4075 50  0000 L CNN
-F 1 "22" H 9925 3975 50  0000 L CNN
-F 2 "Resistor_SMD:R_0603_1608Metric_Pad1.05x0.95mm_HandSolder" V 10005 4025 50  0001 C CNN
-F 3 "~" H 10075 4025 50  0001 C CNN
-	1    10075 4025
+P 10075 4625
+F 0 "R14" H 9875 4675 50  0000 L CNN
+F 1 "22" H 9925 4575 50  0000 L CNN
+F 2 "Resistor_SMD:R_0603_1608Metric_Pad1.05x0.95mm_HandSolder" V 10005 4625 50  0001 C CNN
+F 3 "~" H 10075 4625 50  0001 C CNN
+	1    10075 4625
 	1    0    0    -1
 $EndComp
@@
 L Device:R R15
 U 1 1 5C1BC400
-P 10200 4025
-F 0 "R15" H 10270 4071 50  0000 L CNN
-F 1 "22" H 10270 3980 50  0000 L CNN
-F 2 "Resistor_SMD:R_0603_1608Metric_Pad1.05x0.95mm_HandSolder" V 10130 4025 50  0001 C CNN
-F 3 "~" H 10200 4025 50  0001 C CNN
-	1    10200 4025
+P 10200 4625
+F 0 "R15" H 10270 4671 50  0000 L CNN
+F 1 "22" H 10270 4580 50  0000 L CNN
+F 2 "Resistor_SMD:R_0603_1608Metric_Pad1.05x0.95mm_HandSolder" V 10130 4625 50  0001 C CNN
+F 3 "~" H 10200 4625 50  0001 C CNN
+	1    10200 4625
 	1    0    0    -1
 $EndComp
@@
 	9175 4400 9775 4400
 Wire Wire Line
-	10075 4400 10075 4975
-Wire Wire Line
-	10075 4400 10075 4175
+	5575 7300 6075 7300
+Wire Wire Line
+	5275 7425 6075 7425
+Text GLabel 6250 1150 2    50   BiDi ~ 0
+P0.12_SCL
+Text GLabel 6250 1050 2    50   BiDi ~ 0
+P0.11_SDA
+Wire Wire Line
+	10075 4975 10075 4775
+Wire Wire Line
+	10200 5100 10200 4775
+Wire Wire Line
+	10075 3600 10075 4400
 Connection ~ 10075 4400
 Wire Wire Line
-	10200 4175 10200 5100
-Wire Wire Line
-	10075 3600 10075 3875
-Wire Wire Line
-	10200 3500 10200 3875
-Wire Wire Line
-	5575 7300 6075 7300
-Wire Wire Line
-	5275 7425 6075 7425
-Wire Wire Line
-	8900 1175 8900 1525
-Wire Wire Line
-	9600 1075 9600 1525
+	10075 4400 10075 4475
+Wire Wire Line
+	10200 3500 10200 4475
+Wire Wire Line
+	8425 1275 8775 1275
+Connection ~ 8425 1275
+Text GLabel 10550 1275 2    50   BiDi ~ 0
+P0.04
+Text GLabel 9550 1275 0    50   BiDi ~ 0
+P0.05
+Wire Wire Line
+	9725 1475 9725 1275
+Wire Wire Line
+	9725 1275 9550 1275
+Wire Wire Line
+	10425 1475 10425 1275
+Wire Wire Line
+	10425 1275 10550 1275
 $EndSCHEMATC

Commit message: Updating rescue lib for NRF52 Reference.
Parts:
- SW1, SW2: symbol Project_Libary:SW_SPST_4pin -> NRF52832_Reference-rescue:SW_SPST_4pin-Project_Libary
- U5: symbol Project_Libary:TCN75AVUA713 -> NRF52832_Reference-rescue:TCN75AVUA713-Project_Libary
Changed lines of the file:
@@
 $EndComp
 $Comp
-L Project_Libary:TCN75AVUA713 U5
+L NRF52832_Reference-rescue:TCN75AVUA713-Project_Libary U5
 U 1 1 5C09FD2C
 P 4425 6500
@@
 	8500 3900 8875 3900
 $Comp
-L Project_Libary:SW_SPST_4pin SW1
+L NRF52832_Reference-rescue:SW_SPST_4pin-Project_Libary SW1
 U 1 1 5C1A448E
 P 8075 1575
@@
 	8125 1275 8425 1275
 $Comp
-L Project_Libary:SW_SPST_4pin SW2
+L NRF52832_Reference-rescue:SW_SPST_4pin-Project_Libary SW2
 U 1 1 5C1A47AD
 P 8925 4200
