File: 18650_charger/18650_charger.sch (KiCad schematic (older format))
At the start: 11 parts

Commit message: Progress on charging circuit.
Parts:
- added C?: 0.1u, symbol Device:C
- added C?: 10u, symbol Device:C
- added F?: Fuse_1A, symbol Device:Fuse_Small
- added J?: Conn_01x02_Male, symbol Connector:Conn_01x02_Male
- added R?: 2k, symbol Device:R
- C?: value C -> 10u
- F?: value Fuse_Small -> Fuse_1A
- R?: value R -> 2k
Connections:
- wire segments 29 -> 65
- no-connect marks 0 -> 6
Other:
- moved on the sheet: D?

Commit message: Added new charging ICs and STM32 MCU for voltage measurement.
Parts:
- removed C? (x2): 10u, symbol Device:C
- removed C?: 0.1u, symbol Device:C
- removed D? (x2): D, symbol Device:D
- removed F? (x2): Fuse_1A, symbol Device:Fuse_Small
- removed J?: USB_B_Micro, symbol Connector:USB_B_Micro
- removed J?: Conn_01x02_Male, symbol Connector:Conn_01x02_Male
- removed R? (x2): R, symbol Device:R
- removed R? (x2): 2k, symbol Device:R
- removed U?: TP4056E-SN2L1P, symbol Project_Libary:TP4056E-SN2L1P
- removed U?: DW01, symbol Project_Libary:DW01
- removed U?: FS8205A, symbol Project_Libary:FS8205A
- added C?: 1uF, symbol Device:C
- added C?: 0.1uF, symbol Device:C
- added D?: LED, symbol Device:LED
- added F?: Fuse, symbol Device:Fuse
- added H? (x2): MountingHole_Pad, symbol Mechanical:MountingHole_Pad
- added J?: USB_C_Receptacle, symbol Connector:USB_C_Receptacle
- added J?: Conn_01x02_Male, symbol Connector:Conn_01x02_Male
- added R?: 2.7k, symbol Device:R_US
- added R?: R_US, symbol Device:R_US
- added R?: 330, symbol Device:R_US
- added R?: 1k, symbol Device:R_US
- added R?: 10k, symbol Device:R_US
- added U?: AP9101CAK6-BVTRG1, symbol Project_Libary:AP9101CAK6-BVTRG1
- added U?: BQ21040DBVR, symbol Project_Libary:BQ21040DBVR
- added U?: DMN2019UTS-13, symbol Project_Libary:DMN2019UTS-13
Connections:
- net labels added: GND, Vbatt+, Vbatt-
- net labels removed: GNDREF
- wire segments 65 -> 53
- no-connect marks 6 -> 12
Other:
- note added: "Fixed 10k resistor between TS and ground disables temp sense function"
- note added: "Rset is 1k ohm for 540mA charge current.\nRset = 540/Iset"

Commit message: Updates to MCU circuit
Parts:
- added Q?: Q_PMOS_GSD, symbol Device:Q_PMOS_GSD
- added R?: 0, symbol Device:R_US
- U?: symbol Project_Libary:AP9101CAK6-BVTRG1 -> 18650_charger-rescue:AP9101CAK6-BVTRG1-Project_Libary
- U?: symbol Project_Libary:BQ21040DBVR -> 18650_charger-rescue:BQ21040DBVR-Project_Libary
- U?: symbol Project_Libary:DMN2019UTS-13 -> 18650_charger-rescue:DMN2019UTS-13-Project_Libary
Connections:
- wire segments 53 -> 65
Other:
- moved on the sheet: C?, F?, H?, J?
Changed lines of the file:
@@
 $EndDescr
 $Comp
-L Project_Libary:AP9101CAK6-BVTRG1 U?
+L 18650_charger-rescue:AP9101CAK6-BVTRG1-Project_Libary U?
 U 1 1 5F25D898
 P 6850 4350
@@
 $EndComp
 $Comp
-L Project_Libary:BQ21040DBVR U?
+L 18650_charger-rescue:BQ21040DBVR-Project_Libary U?
 U 1 1 5F25DC0D
 P 4950 3950
@@
 $EndComp
 $Comp
-L Project_Libary:DMN2019UTS-13 U?
+L 18650_charger-rescue:DMN2019UTS-13-Project_Libary U?
 U 1 1 5F25DF53
 P 6850 5250
@@
 L Connector:USB_C_Receptacle J?
 U 1 1 5F267AF4
-P 2200 4800
-F 0 "J?" H 2307 6067 50  0000 C CNN
-F 1 "USB_C_Receptacle" H 2307 5976 50  0000 C CNN
-F 2 "" H 2350 4800 50  0001 C CNN
-F 3 "https://www.usb.org/sites/default/files/documents/usb_type-c.zip" H 2350 4800 50  0001 C CNN
-	1    2200 4800
-	1    0    0    -1
-$EndComp
-$Comp
-L Device:Fuse F?
-U 1 1 5F26A8E6
-P 3600 3850
-F 0 "F?" V 3403 3850 50  0000 C CNN
-F 1 "Fuse" V 3494 3850 50  0000 C CNN
-F 2 "" V 3530 3850 50  0001 C CNN
-F 3 "~" H 3600 3850 50  0001 C CNN
-	1    3600 3850
-	0    1    1    0
+P 2050 4850
+F 0 "J?" H 2157 6117 50  0000 C CNN
+F 1 "USB_C_Receptacle" H 2157 6026 50  0000 C CNN
+F 2 "" H 2200 4850 50  0001 C CNN
+F 3 "https://www.usb.org/sites/default/files/documents/usb_type-c.zip" H 2200 4850 50  0001 C CNN
+	1    2050 4850
+	1    0    0    -1
 $EndComp
 $Comp
@@
 L Device:C C?
 U 1 1 5F26EE17
-P 3950 4000
-F 0 "C?" H 4065 4046 50  0000 L CNN
-F 1 "1uF" H 4065 3955 50  0000 L CNN
-F 2 "" H 3988 3850 50  0001 C CNN
-F 3 "~" H 3950 4000 50  0001 C CNN
-	1    3950 4000
+P 3950 4150
+F 0 "C?" H 4065 4196 50  0000 L CNN
+F 1 "1uF" H 4065 4105 50  0000 L CNN
+F 2 "" H 3988 4000 50  0001 C CNN
+F 3 "~" H 3950 4150 50  0001 C CNN
+	1    3950 4150
 	1    0    0    -1
 $EndComp
@@
 L Mechanical:MountingHole_Pad H?
 U 1 1 5F264E8A
-P 3200 3350
-F 0 "H?" H 3300 3399 50  0000 L CNN
-F 1 "MountingHole_Pad" H 3300 3308 50  0000 L CNN
-F 2 "" H 3200 3350 50  0001 C CNN
-F 3 "~" H 3200 3350 50  0001 C CNN
-	1    3200 3350
+P 2800 3150
+F 0 "H?" H 2900 3199 50  0000 L CNN
+F 1 "MountingHole_Pad" H 2900 3108 50  0000 L CNN
+F 2 "" H 2800 3150 50  0001 C CNN
+F 3 "~" H 2800 3150 50  0001 C CNN
+	1    2800 3150
 	1    0    0    -1
 $EndComp
@@
 Text Notes 800  900  0    50   ~ 0
 Rset is 1k ohm for 540mA charge current.\nRset = 540/Iset
-NoConn ~ 2800 5800
-NoConn ~ 2800 5700
-NoConn ~ 2800 5500
-NoConn ~ 2800 5400
-NoConn ~ 2800 5200
-NoConn ~ 2800 5100
-NoConn ~ 2800 4900
-NoConn ~ 2800 4800
-NoConn ~ 2800 4600
-NoConn ~ 2800 4500
-NoConn ~ 2800 4400
-NoConn ~ 2800 4300
+NoConn ~ 2650 5850
+NoConn ~ 2650 5750
+NoConn ~ 2650 5550
+NoConn ~ 2650 5450
+NoConn ~ 2650 5250
+NoConn ~ 2650 5150
+NoConn ~ 2650 4950
+NoConn ~ 2650 4850
+NoConn ~ 2650 4650
+NoConn ~ 2650 4550
+NoConn ~ 2650 4450
+NoConn ~ 2650 4350
 Text Notes 800  1100 0    50   ~ 0
 Fixed 10k resistor between TS and ground disables temp sense function
@@
 	3750 3850 3950 3850
 Wire Wire Line
-	3950 3850 4600 3850
-Connection ~ 3950 3850
-Wire Wire Line
 	4600 3950 4300 3950
 Wire Wire Line
@@
 Wire Wire Line
 	4600 4500 4600 4050
-Wire Wire Line
-	3950 4150 3950 4500
 Wire Wire Line
 	3950 4500 4300 4500
@@
 Wire Wire Line
 	7450 5200 8350 5200
-$Sheet
-S 6300 2000 1100 1000
-U 5F318FD2
-F0 "Voltage measurement" 50
-F1 "Voltage measurement.sch" 50
-$EndSheet
 Text HLabel 8550 3850 2    50   Input ~ 0
 Vbatt+
@@
 	8600 5200 8350 5200
 Connection ~ 8350 5200
+$Sheet
+S 4700 2300 1100 1000
+U 5F318FD2
+F0 "Voltage measurement" 50
+F1 "Voltage measurement.sch" 50
+F2 "Vbatt+" I R 5800 2450 50
+F3 "Vbatt-" U R 5800 2600 50
+F4 "USB_+5V" I L 4700 2450 50
+F5 "Charge_Ctrl" I L 4700 2600 50
+$EndSheet
+$Comp
+L Device:Fuse F?
+U 1 1 5F26A8E6
+P 3400 3850
+F 0 "F?" V 3203 3850 50  0000 C CNN
+F 1 "Fuse" V 3294 3850 50  0000 C CNN
+F 2 "" V 3330 3850 50  0001 C CNN
+F 3 "~" H 3400 3850 50  0001 C CNN
+	1    3400 3850
+	0    1    1    0
+$EndComp
+Wire Wire Line
+	3950 3850 3950 4000
+Wire Wire Line
+	3950 4500 3950 4300
+Wire Wire Line
+	4050 3850 3950 3850
+Connection ~ 3950 3850
+Wire Wire Line
+	4450 3850 4600 3850
+Wire Wire Line
+	3750 3850 3750 3550
+Wire Wire Line
+	3750 3550 3850 3550
+Wire Wire Line
+	3550 3850 3750 3850
+Connection ~ 3750 3850
+$Comp
+L Device:R_US R?
+U 1 1 5F43F0EE
+P 4250 3150
+F 0 "R?" H 4318 3196 50  0000 L CNN
+F 1 "0" H 4318 3105 50  0000 L CNN
+F 2 "" V 4290 3140 50  0001 C CNN
+F 3 "~" H 4250 3150 50  0001 C CNN
+	1    4250 3150
+	1    0    0    -1
+$EndComp
+Wire Wire Line
+	4250 2600 4700 2600
+Wire Wire Line
+	4250 2600 4250 3000
+Wire Wire Line
+	3750 3550 3750 2450
+Wire Wire Line
+	3750 2450 4700 2450
+Connection ~ 3750 3550
+Wire Wire Line
+	5800 2450 6100 2450
+Wire Wire Line
+	5800 2600 6100 2600
+Text HLabel 6100 2450 2    50   Input ~ 0
+Vbatt+
+Text HLabel 6100 2600 2    50   Input ~ 0
+Vbatt-
+Wire Wire Line
+	3250 3850 2650 3850
+$Comp
+L Device:Q_PMOS_GSD Q?
+U 1 1 5F42065E
+P 4250 3750
+F 0 "Q?" V 4150 3900 50  0000 C CNN
+F 1 "Q_PMOS_GSD" V 4050 4100 50  0000 C CNN
+F 2 "" H 4450 3850 50  0001 C CNN
+F 3 "~" H 4250 3750 50  0001 C CNN
+	1    4250 3750
+	0    1    1    0
+$EndComp
 $EndSCHEMATC

Commit message: Update to MCU circuit
Parts:
- removed H? (x2): MountingHole_Pad, symbol Mechanical:MountingHole_Pad
- added C?: NC, symbol Device:C
- added R?: 1k, symbol Device:R_US
- added R?: 0, symbol Device:R_US
Connections:
- net GND is gone; now on net GND1: C?.2, R?.2, R?.2, R?.2, U?.2 (S1), U?.3 (S1), U?.5 (GND)
- net Voltage measurement/USB_+5V: now also R?.1
- net GND1: now reaches J?.A1 (GND), J?.A12 (GND), J?.B1 (GND), J?.B12 (GND)
- net GND1: now also C?.2, R?.2
- net at J?.S1 (SHIELD): now also C?.1, R?.1
- net at Q?.1 (G): now also R?.2, R?.2
Changed lines of the file:
@@
-	1    0    0    -1
-$EndComp
-$Comp
-L power:GND #PWR?
-U 1 1 5F2B416F
-P 4600 4550
-F 0 "#PWR?" H 4600 4300 50  0001 C CNN
-F 1 "GND" H 4605 4377 50  0000 C CNN
-F 2 "" H 4600 4550 50  0001 C CNN
-F 3 "" H 4600 4550 50  0001 C CNN
-	1    4600 4550
-	1    0    0    -1
-$EndComp
-$Comp
-L power:GND #PWR?
-U 1 1 5F2B46B1
-P 6100 5550
-F 0 "#PWR?" H 6100 5300 50  0001 C CNN
-F 1 "GND" H 6105 5377 50  0000 C CNN
-F 2 "" H 6100 5550 50  0001 C CNN
-F 3 "" H 6100 5550 50  0001 C CNN
-	1    6100 5550
-	1    0    0    -1
-$EndComp
-$Comp
-L Mechanical:MountingHole_Pad H?
-U 1 1 5F264E8A
-P 2800 3150
-F 0 "H?" H 2900 3199 50  0000 L CNN
-F 1 "MountingHole_Pad" H 2900 3108 50  0000 L CNN
-F 2 "" H 2800 3150 50  0001 C CNN
-F 3 "~" H 2800 3150 50  0001 C CNN
-	1    2800 3150
-	1    0    0    -1
-$EndComp
-$Comp
-L Mechanical:MountingHole_Pad H?
-U 1 1 5F26662E
-P 2450 7050
-F 0 "H?" H 2550 7099 50  0000 L CNN
-F 1 "MountingHole_Pad" H 2550 7008 50  0000 L CNN
-F 2 "" H 2450 7050 50  0001 C CNN
-F 3 "~" H 2450 7050 50  0001 C CNN
-	1    2450 7050
 	1    0    0    -1
 $EndComp
@@
 	0    1    1    0
 $EndComp
+$Comp
+L Device:R_US R?
+U 1 1 5F3A1849
+P 4000 3550
+F 0 "R?" V 4050 3650 50  0000 L CNN
+F 1 "1k" V 4050 3350 50  0000 L CNN
+F 2 "" V 4040 3540 50  0001 C CNN
+F 3 "~" H 4000 3550 50  0001 C CNN
+	1    4000 3550
+	0    -1   -1   0
+$EndComp
+Wire Wire Line
+	4150 3550 4250 3550
+Wire Wire Line
+	4250 3300 4250 3550
+Connection ~ 4250 3550
+$Comp
+L power:GND1 #PWR?
+U 1 1 5F3D1CA0
+P 4600 4550
+F 0 "#PWR?" H 4600 4300 50  0001 C CNN
+F 1 "GND1" H 4605 4377 50  0000 C CNN
+F 2 "" H 4600 4550 50  0001 C CNN
+F 3 "" H 4600 4550 50  0001 C CNN
+	1    4600 4550
+	1    0    0    -1
+$EndComp
+$Comp
+L power:GND1 #PWR?
+U 1 1 5F3D255E
+P 6100 5550
+F 0 "#PWR?" H 6100 5300 50  0001 C CNN
+F 1 "GND1" H 6105 5377 50  0000 C CNN
+F 2 "" H 6100 5550 50  0001 C CNN
+F 3 "" H 6100 5550 50  0001 C CNN
+	1    6100 5550
+	1    0    0    -1
+$EndComp
+$Comp
+L power:GND1 #PWR?
+U 1 1 5F3D2AF9
+P 2050 6950
+F 0 "#PWR?" H 2050 6700 50  0001 C CNN
+F 1 "GND1" H 2055 6777 50  0000 C CNN
+F 2 "" H 2050 6950 50  0001 C CNN
+F 3 "" H 2050 6950 50  0001 C CNN
+	1    2050 6950
+	1    0    0    -1
+$EndComp
+$Comp
+L Device:R_US R?
+U 1 1 5F3D37C0
+P 1750 6700
+F 0 "R?" H 1818 6746 50  0000 L CNN
+F 1 "0" H 1818 6655 50  0000 L CNN
+F 2 "" V 1790 6690 50  0001 C CNN
+F 3 "~" H 1750 6700 50  0001 C CNN
+	1    1750 6700
+	1    0    0    -1
+$EndComp
+$Comp
+L Device:C C?
+U 1 1 5F3D5BC2
+P 1450 6700
+F 0 "C?" H 1565 6746 50  0000 L CNN
+F 1 "NC" H 1565 6655 50  0000 L CNN
+F 2 "" H 1488 6550 50  0001 C CNN
+F 3 "~" H 1450 6700 50  0001 C CNN
+	1    1450 6700
+	1    0    0    -1
+$EndComp
+Wire Wire Line
+	1450 6550 1750 6550
+Wire Wire Line
+	1750 6550 1750 6450
+Connection ~ 1750 6550
+Wire Wire Line
+	1450 6850 1750 6850
+Wire Wire Line
+	1750 6850 2050 6850
+Wire Wire Line
+	2050 6850 2050 6950
+Connection ~ 1750 6850
+Wire Wire Line
+	2050 6450 2050 6850
+Connection ~ 2050 6850
 $EndSCHEMATC
