File: 18650_charger/Voltage measurement.sch (KiCad schematic (older format))
At the start: 20 parts

Commit message: Updates to MCU circuit
Parts:
- removed R? (x7): R_US, symbol Device:R_US
- added C? (x5): C, symbol Device:C
- added D? (x2): D, symbol Device:D
- added D?: LED, symbol Device:LED
- added J?: Conn_01x05_Female, symbol Connector:Conn_01x05_Female
- added R? (x6): R_US, symbol Device:R_US
- added R?: 330, symbol Device:R_US
- U?: symbol Project_Libary:BC56-12SRWA -> 18650_charger-rescue:BC56-12SRWA-Project_Libary
- U? (x2): symbol Project_Libary:DMN63D8LDW-7 -> 18650_charger-rescue:DMN63D8LDW-7-Project_Libary
- U?: symbol Project_Libary:REG711EA-3.3_250 -> 18650_charger-rescue:REG711EA-3.3_250-Project_Libary
Connections:
- net labels added: +3.3V, BOOT0, DIGIT_1, DIGIT_2, DIGIT_3, GND, RX, TX, USB_+5V, Vbatt+
- wire segments 0 -> 89
Other:
- moved on the sheet: C?, R?

Commit message: Update to MCU circuit
Parts:
- added J?: Conn_01x03_Female, symbol Connector:Conn_01x03_Female
- added Q?: Q_NMOS_GSD, symbol Device:Q_NMOS_GSD
- added R?: 1k, symbol Device:R_US
- added SW?: SW_Push, symbol Switch:SW_Push
- C?: value C -> 0.22uF
- C? (x2): value C -> 2.2uF
- J?: symbol Connector:Conn_01x05_Female -> Connector:Conn_01x04_Female
Connections:
- net labels added: Charge_Ctrl, GND2, Vbatt-
- net labels removed: GND
- wire segments 89 -> 101
Changed lines of the file:
@@
 P 5700 7100
 F 0 "C?" H 5815 7146 50  0000 L CNN
-F 1 "C" H 5815 7055 50  0000 L CNN
+F 1 "0.22uF" H 5815 7055 50  0000 L CNN
 F 2 "" H 5738 6950 50  0001 C CNN
 F 3 "~" H 5700 7100 50  0001 C CNN
@@
 P 4050 6950
 F 0 "C?" H 4165 6996 50  0000 L CNN
-F 1 "C" H 4165 6905 50  0000 L CNN
+F 1 "2.2uF" H 4165 6905 50  0000 L CNN
 F 2 "" H 4088 6800 50  0001 C CNN
 F 3 "~" H 4050 6950 50  0001 C CNN
@@
 P 6150 6950
 F 0 "C?" H 6265 6996 50  0000 L CNN
-F 1 "C" H 6265 6905 50  0000 L CNN
+F 1 "2.2uF" H 6265 6905 50  0000 L CNN
 F 2 "" H 6188 6800 50  0001 C CNN
 F 3 "~" H 6150 6950 50  0001 C CNN
@@
 Wire Wire Line
 	4450 6800 4050 6800
-$Comp
-L power:GND #PWR?
-U 1 1 5F3ACD87
-P 4450 7300
-F 0 "#PWR?" H 4450 7050 50  0001 C CNN
-F 1 "GND" H 4455 7127 50  0000 C CNN
-F 2 "" H 4450 7300 50  0001 C CNN
-F 3 "" H 4450 7300 50  0001 C CNN
-	1    4450 7300
-	1    0    0    -1
-$EndComp
-$Comp
-L power:GND #PWR?
-U 1 1 5F3AE2DB
-P 6150 7300
-F 0 "#PWR?" H 6150 7050 50  0001 C CNN
-F 1 "GND" H 6155 7127 50  0000 C CNN
-F 2 "" H 6150 7300 50  0001 C CNN
-F 3 "" H 6150 7300 50  0001 C CNN
-	1    6150 7300
-	1    0    0    -1
-$EndComp
 Wire Wire Line
 	4550 7050 4450 7050
@@
 	7850 1600 7850 1350
 Connection ~ 7850 1600
-$Comp
-L power:GND #PWR?
-U 1 1 5F3B4471
-P 7850 2500
-F 0 "#PWR?" H 7850 2250 50  0001 C CNN
-F 1 "GND" H 7855 2327 50  0000 C CNN
-F 2 "" H 7850 2500 50  0001 C CNN
-F 3 "" H 7850 2500 50  0001 C CNN
-	1    7850 2500
-	1    0    0    -1
-$EndComp
-$Comp
-L power:GND #PWR?
-U 1 1 5F3B54BA
-P 5950 5350
-F 0 "#PWR?" H 5950 5100 50  0001 C CNN
-F 1 "GND" H 5955 5177 50  0000 C CNN
-F 2 "" H 5950 5350 50  0001 C CNN
-F 3 "" H 5950 5350 50  0001 C CNN
-	1    5950 5350
-	1    0    0    -1
-$EndComp
 Wire Wire Line
 	7500 1900 7850 1900
@@
 	5650 5250 5750 5250
 Connection ~ 5750 5250
-$Comp
-L Connector:Conn_01x05_Female J?
-U 1 1 5F3BC82B
-P 1150 4650
-F 0 "J?" H 1042 5035 50  0000 C CNN
-F 1 "Conn_01x05_Female" H 1042 4944 50  0000 C CNN
-F 2 "" H 1150 4650 50  0001 C CNN
-F 3 "~" H 1150 4650 50  0001 C CNN
-	1    1150 4650
-	-1   0    0    -1
-$EndComp
-Wire Wire Line
-	1350 4450 1850 4450
-Wire Wire Line
-	1350 4550 1850 4550
-Wire Wire Line
-	1350 4650 1850 4650
-Wire Wire Line
-	1350 4750 1850 4750
-Wire Wire Line
-	1350 4850 1850 4850
+Wire Wire Line
+	1400 4150 1900 4150
+Wire Wire Line
+	1400 4250 1900 4250
+Wire Wire Line
+	1400 4350 1900 4350
 Wire Wire Line
 	8900 2900 9350 2900
@@
 Text HLabel 10050 3100 2    50   Input ~ 0
 DIGIT_1
-Text HLabel 1850 4850 2    50   Input ~ 0
+Text HLabel 1900 3450 2    50   Input ~ 0
 BOOT0
-Text HLabel 1850 4750 2    50   Input ~ 0
-GND
-Text HLabel 1850 4650 2    50   Input ~ 0
+Text HLabel 1900 4350 2    50   Input ~ 0
 RX
-Text HLabel 1850 4550 2    50   Input ~ 0
+Text HLabel 1900 4250 2    50   Input ~ 0
 TX
-$Comp
-L power:GND #PWR?
-U 1 1 5F3E8808
-P 9200 4700
-F 0 "#PWR?" H 9200 4450 50  0001 C CNN
-F 1 "GND" H 9205 4527 50  0000 C CNN
-F 2 "" H 9200 4700 50  0001 C CNN
-F 3 "" H 9200 4700 50  0001 C CNN
-	1    9200 4700
-	1    0    0    -1
-$EndComp
-$Comp
-L power:GND #PWR?
-U 1 1 5F3E9685
-P 10200 4700
-F 0 "#PWR?" H 10200 4450 50  0001 C CNN
-F 1 "GND" H 10205 4527 50  0000 C CNN
-F 2 "" H 10200 4700 50  0001 C CNN
-F 3 "" H 10200 4700 50  0001 C CNN
-	1    10200 4700
-	1    0    0    -1
-$EndComp
-$Comp
-L power:GND #PWR?
-U 1 1 5F3E9C8E
-P 9200 5350
-F 0 "#PWR?" H 9200 5100 50  0001 C CNN
-F 1 "GND" H 9205 5177 50  0000 C CNN
-F 2 "" H 9200 5350 50  0001 C CNN
-F 3 "" H 9200 5350 50  0001 C CNN
-	1    9200 5350
-	1    0    0    -1
-$EndComp
 Wire Wire Line
 	9200 4700 9200 4650
@@
 Wire Wire Line
 	10200 4650 10000 4650
-$Comp
-L power:GND #PWR?
-U 1 1 5F3EF5F0
-P 10200 5350
-F 0 "#PWR?" H 10200 5100 50  0001 C CNN
-F 1 "GND" H 10205 5177 50  0000 C CNN
-F 2 "" H 10200 5350 50  0001 C CNN
-F 3 "" H 10200 5350 50  0001 C CNN
-	1    10200 5350
-	1    0    0    -1
-$EndComp
 Wire Wire Line
 	10000 5300 10100 5300
@@
 Wire Wire Line
 	4050 6500 4050 6800
-Text HLabel 1850 4450 2    50   Input ~ 0
+Text HLabel 1900 4150 2    50   Input ~ 0
 +3.3V
 Text HLabel 6400 6800 2    50   Input ~ 0
@@
 Wire Wire Line
 	8250 1600 7850 1600
+$Comp
+L Device:Q_NMOS_GSD Q?
+U 1 1 5F3A7C05
+P 1550 5600
+F 0 "Q?" H 1755 5646 50  0000 L CNN
+F 1 "Q_NMOS_GSD" H 1755 5555 50  0000 L CNN
+F 2 "" H 1750 5700 50  0001 C CNN
+F 3 "~" H 1550 5600 50  0001 C CNN
+	1    1550 5600
+	-1   0    0    -1
+$EndComp
+$Comp
+L Device:R_US R?
+U 1 1 5F3AB44F
+P 2100 5600
+F 0 "R?" V 2150 5700 50  0000 L CNN
+F 1 "1k" V 2150 5350 50  0000 L CNN
+F 2 "" V 2140 5590 50  0001 C CNN
+F 3 "~" H 2100 5600 50  0001 C CNN
+	1    2100 5600
+	0    -1   -1   0
+$EndComp
+Text HLabel 1450 5200 0    50   Input ~ 0
+Charge_Ctrl
+Wire Wire Line
+	1450 5400 1450 5200
+Wire Wire Line
+	1450 6000 1450 5800
+Wire Wire Line
+	1750 5600 1950 5600
+Text HLabel 3350 7150 0    50   Input ~ 0
+Vbatt-
+Wire Wire Line
+	3350 7150 4050 7150
+Connection ~ 4050 7150
+$Comp
+L power:GND2 #PWR?
+U 1 1 5F3CA84C
+P 1450 6000
+F 0 "#PWR?" H 1450 5750 50  0001 C CNN
+F 1 "GND2" H 1455 5827 50  0000 C CNN
+F 2 "" H 1450 6000 50  0001 C CNN
+F 3 "" H 1450 6000 50  0001 C CNN
+	1    1450 6000
+	1    0    0    -1
+$EndComp
+$Comp
+L power:GND2 #PWR?
+U 1 1 5F3CBC36
+P 4450 7300
+F 0 "#PWR?" H 4450 7050 50  0001 C CNN
+F 1 "GND2" H 4455 7127 50  0000 C CNN
+F 2 "" H 4450 7300 50  0001 C CNN
+F 3 "" H 4450 7300 50  0001 C CNN
+	1    4450 7300
+	1    0    0    -1
+$EndComp
+$Comp
+L power:GND2 #PWR?
+U 1 1 5F3CC22E
+P 6150 7300
+F 0 "#PWR?" H 6150 7050 50  0001 C CNN
+F 1 "GND2" H 6155 7127 50  0000 C CNN
+F 2 "" H 6150 7300 50  0001 C CNN
+F 3 "" H 6150 7300 50  0001 C CNN
+	1    6150 7300
+	1    0    0    -1
+$EndComp
+$Comp
+L power:GND2 #PWR?
+U 1 1 5F3CC74C
+P 9200 5350
+F 0 "#PWR?" H 9200 5100 50  0001 C CNN
+F 1 "GND2" H 9205 5177 50  0000 C CNN
+F 2 "" H 9200 5350 50  0001 C CNN
+F 3 "" H 9200 5350 50  0001 C CNN
+	1    9200 5350
+	1    0    0    -1
+$EndComp
+$Comp
+L power:GND2 #PWR?
+U 1 1 5F3CCD0A
+P 9200 4700
+F 0 "#PWR?" H 9200 4450 50  0001 C CNN
+F 1 "GND2" H 9205 4527 50  0000 C CNN
+F 2 "" H 9200 4700 50  0001 C CNN
+F 3 "" H 9200 4700 50  0001 C CNN
+	1    9200 4700
+	1    0    0    -1
+$EndComp
+$Comp
+L power:GND2 #PWR?
+U 1 1 5F3CD0B5
+P 10200 4700
+F 0 "#PWR?" H 10200 4450 50  0001 C CNN
+F 1 "GND2" H 10205 4527 50  0000 C CNN
+F 2 "" H 10200 4700 50  0001 C CNN
+F 3 "" H 10200 4700 50  0001 C CNN
+	1    10200 4700
+	1    0    0    -1
+$EndComp
+$Comp
+L power:GND2 #PWR?
+U 1 1 5F3CD53A
+P 10200 5350
+F 0 "#PWR?" H 10200 5100 50  0001 C CNN
+F 1 "GND2" H 10205 5177 50  0000 C CNN
+F 2 "" H 10200 5350 50  0001 C CNN
+F 3 "" H 10200 5350 50  0001 C CNN
+	1    10200 5350
+	1    0    0    -1
+$EndComp
+$Comp
+L power:GND2 #PWR?
+U 1 1 5F3CD859
+P 5950 5350
+F 0 "#PWR?" H 5950 5100 50  0001 C CNN
+F 1 "GND2" H 5955 5177 50  0000 C CNN
+F 2 "" H 5950 5350 50  0001 C CNN
+F 3 "" H 5950 5350 50  0001 C CNN
+	1    5950 5350
+	1    0    0    -1
+$EndComp
+$Comp
+L power:GND2 #PWR?
+U 1 1 5F3CE020
+P 7850 2500
+F 0 "#PWR?" H 7850 2250 50  0001 C CNN
+F 1 "GND2" H 7855 2327 50  0000 C CNN
+F 2 "" H 7850 2500 50  0001 C CNN
+F 3 "" H 7850 2500 50  0001 C CNN
+	1    7850 2500
+	1    0    0    -1
+$EndComp
+$Comp
+L power:GND2 #PWR?
+U 1 1 5F3CE8DF
+P 1950 4550
+F 0 "#PWR?" H 1950 4300 50  0001 C CNN
+F 1 "GND2" H 1955 4377 50  0000 C CNN
+F 2 "" H 1950 4550 50  0001 C CNN
+F 3 "" H 1950 4550 50  0001 C CNN
+	1    1950 4550
+	1    0    0    -1
+$EndComp
+$Comp
+L Connector:Conn_01x04_Female J?
+U 1 1 5F3BC82B
+P 1200 4250
+F 0 "J?" H 1092 4635 50  0000 C CNN
+F 1 "Conn_01x05_Female" H 1092 4544 50  0000 C CNN
+F 2 "" H 1200 4250 50  0001 C CNN
+F 3 "~" H 1200 4250 50  0001 C CNN
+	1    1200 4250
+	-1   0    0    -1
+$EndComp
+Wire Wire Line
+	1400 4450 1950 4450
+Wire Wire Line
+	1950 4450 1950 4550
+$Comp
+L Connector:Conn_01x03_Female J?
+U 1 1 5F3F2C40
+P 1200 3450
+F 0 "J?" H 1092 3735 50  0000 C CNN
+F 1 "Conn_01x03_Female" H 1092 3644 50  0000 C CNN
+F 2 "" H 1200 3450 50  0001 C CNN
+F 3 "~" H 1200 3450 50  0001 C CNN
+	1    1200 3450
+	-1   0    0    -1
+$EndComp
+Text HLabel 1900 3350 2    50   Input ~ 0
++3.3V
+$Comp
+L power:GND2 #PWR?
+U 1 1 5F3F4E62
+P 1950 3600
+F 0 "#PWR?" H 1950 3350 50  0001 C CNN
+F 1 "GND2" H 1955 3427 50  0000 C CNN
+F 2 "" H 1950 3600 50  0001 C CNN
+F 3 "" H 1950 3600 50  0001 C CNN
+	1    1950 3600
+	1    0    0    -1
+$EndComp
+Wire Wire Line
+	1900 3450 1400 3450
+Wire Wire Line
+	1900 3350 1400 3350
+$Comp
+L Switch:SW_Push SW?
+U 1 1 5F3FEC11
+P 4800 2350
+F 0 "SW?" H 4800 2635 50  0000 C CNN
+F 1 "SW_Push" H 4800 2544 50  0000 C CNN
+F 2 "" H 4800 2550 50  0001 C CNN
+F 3 "~" H 4800 2550 50  0001 C CNN
+	1    4800 2350
+	1    0    0    -1
+$EndComp
+Wire Wire Line
+	5150 2550 4900 2550
+Text HLabel 4900 2550 0    50   Input ~ 0
+BOOT0
+$Comp
+L power:GND2 #PWR?
+U 1 1 5F403222
+P 4350 2400
+F 0 "#PWR?" H 4350 2150 50  0001 C CNN
+F 1 "GND2" H 4355 2227 50  0000 C CNN
+F 2 "" H 4350 2400 50  0001 C CNN
+F 3 "" H 4350 2400 50  0001 C CNN
+	1    4350 2400
+	1    0    0    -1
+$EndComp
+Wire Wire Line
+	4600 2350 4350 2350
+Wire Wire Line
+	4350 2350 4350 2400
+Wire Wire Line
+	5000 2350 5150 2350
+Wire Wire Line
+	1950 3550 1950 3600
+Wire Wire Line
+	1400 3550 1950 3550
 $EndSCHEMATC

Commit message: Updated STM32 schematic
Parts:
- removed D? (x2): D, symbol Device:D
- added C? (x4): 1uF, symbol Device:C
- added C? (x4): NC, symbol Device:C
- added D? (x2): D_Schottky, symbol Device:D_Schottky
- added F?: Fuse, symbol Device:Fuse
- added R?: 0, symbol Device:R_US
- added SW?: SW_DPST, symbol Switch:SW_DPST
- added X? (x2): SG-8002CE, Oscillator:Oscillator_SMD_SeikoEpson_SG8002CE-4Pin_3.2x2.5mm, symbol Oscillator:SG-8002CE
- C?: value C -> 1uF
- C? (x4): value C -> 100nF
Connections:
- net labels added: CHARGE_EN, DIGIT_1_EN, DIGIT_2_EN, DIGIT_3_EN, LED_A, LED_B, LED_C, LED_D, LED_DP, LED_E, LED_F, LED_G, USART1_RX, USART1_TX
- net labels removed: RX, TX
- wire segments 101 -> 166
- no-connect marks 0 -> 19
Other:
- moved on the sheet: C?, D?, R?, U?
